Commit message: a1 lidar changes

File: roomblock_description/robots/roomblock.urdf.xacro (robot description, xacro)
@@ -26,5 +26,5 @@
   </link>
   <joint name="laser_joint" type="fixed">
-    <origin xyz="0 0 0.1308" rpy="0 0 ${M_PI}" />
+    <origin xyz="0 0 0.1308" rpy="0 0 ${M_PI/2}" />
     <parent link="block_link" />
     <child link="laser" />
